File: hw/Stepstick.sch (KiCad schematic (older format))
At the start: 23 parts

Commit message: Added some of the netlist
Parts:
- removed P?: CONN_4, symbol CONN_4
- added P1, P6: CONN_2, symbol CONN_2
- gave numbers to parts that had none: 22
Connections:
- wire segments 108 -> 115
