File: hw/Stepstick.kicad_pcb (KiCad board)
At the start: 2 copper layers, 80 x 61 mm, 41 parts, among them P1 CONN_2, P2 CONN_2, P3 CONN_4, P4 CONN_4, P5 CONN_2, P6 CONN_2, U1 ACS711, U2 StepStick, U3 Jumper_3, U4 Pro_Micro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

Commit message: pcb layout completed
Parts:
- C2, C4, C6, C7, R12, R2, U1, U6, X1: moved to B.Cu
- P2: value CONN_2 -> 12V
- P5: value CONN_2 -> CAN Bus
- moved R2 45.7 mm to (115.5, 88.2)
- moved R3 42.7 mm to (156.2, 97.0), turned to 270 degrees
- moved R8 37.4 mm to (119.2, 88.8)
- moved R1 37.2 mm to (153.0, 97.0), turned to 270 degrees
- moved R12 36.5 mm to (119.2, 91.2), turned to 180 degrees
- moved C4 31.9 mm to (115.5, 91.2)
- moved C1 31.1 mm to (122.5, 88.8), turned to 180 degrees
- moved C5 24.2 mm to (121.0, 102.0), turned to 180 degrees
- moved D1 22.9 mm to (158.0, 90.2), turned to 270 degrees
- moved R4 22.0 mm to (158.0, 93.2), turned to 270 degrees
- moved C7 21.3 mm to (110.8, 108.5), turned to 90 degrees
- moved C3 20.7 mm to (121.2, 82.5)
- moved D2 18.9 mm to (155.0, 90.2), turned to 270 degrees
- moved C6 18.5 mm to (115.8, 108.5), turned to 90 degrees
- moved X1 18.2 mm to (113.2, 104.5), turned to 180 degrees
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- renumbered 3mmHole to 3mmHole_2
Routing:
- net GND: track 0.00 -> 232.0 mm
- net VCC: track 0.00 -> 176.9 mm, vias 0 -> 1
- net /Step: track 0.00 -> 75.4 mm
- net /SCL: track 0.00 -> 75.2 mm, vias 0 -> 1
- net /SDA: track 0.00 -> 60.9 mm
- net /Dir: track 0.00 -> 58.6 mm
- net /Vmot: track 0.00 -> 54.9 mm
- net /MS1: track 0.00 -> 44.4 mm, vias 0 -> 1
- net /MS2: track 0.00 -> 43.2 mm
- net /CAN_Bus/CANL: track 0.00 -> 42.9 mm, vias 0 -> 1
- net /MS3: track 0.00 -> 38.7 mm
- net /CAN_Bus/CANH: track 0.00 -> 38.7 mm
- net /Enable: track 0.00 -> 37.0 mm
- net /Sense_Current: track 0.00 -> 35.4 mm
- net /CAN_Bus/CAN_SCK: track 0.00 -> 35.4 mm
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- added copper zone on B.Cu, net GND
- added copper zone on F.Cu, net GND
Other:
- board size 80 x 61 mm -> 70.2 x 43 mm
- board text added: "1"
- board text added: "10to7.com"
- board text added: "12V"
- board text added: "1A"
- board text added: "1B"
- board text added: "2"
- board text added: "2A"
- board text added: "2B"
- board text added: "3"
- board text added: ": 12 (9/A9) : 5 (2) : 6 (3) : 17 (18/A0) : 10 (7)"
- board text added: ": 2 (0) : 11 (8/A8) : 7 (4/A6) : 8 (5) : 9 (6/A7)"
- board text added: "CAN SCK SO SI CS INT"
- board text added: "Dir"
- board text added: "Enable"
- board text added: "Fault"
- board text added: "Fault LED SDA SCL Current sense Current fault"
- board text added: "GND"
- board text added: "Hi"
- board text added: "Int"
- board text added: "Low"
- board text added: "Pin : 16 (15) : 15 (14) : 14 (16) : 13 (19) : 1(1)"
- board text added: "Pro Micro"
- board text added: "RX"
- board text added: "SCL"
- board text added: "SDA"
- board text added: "Step"
- board text added: "Step Dir MS1 MS2 MS3"
- board text added: "Step Stick"
- board text added: "TX"
- board text added: "USB"
- board text added: "VCC"
